Commit message: Se cambia de posición al robot y se empieza a validar la sujeción del gripper.

File: proyecto_intermedio_robotica/urdf/links_joints.xacro (robot description, xacro)
@@ -68,4 +68,31 @@
     </gazebo>
  </xacro:macro>
+ <xacro:macro name="link_mesh" params="name origin_xyz origin_rpy meshfile mass ixx ixy ixz iyy iyz izz">
+    <link name="${name}">
+      <inertial>
+        <mass value="${mass}" />
+        <origin rpy="${origin_rpy}" xyz="${origin_xyz}" />
+        <inertia ixx="${ixx}" ixy="${ixy}" ixz="${ixz}" iyy="${iyy}" iyz="${iyz}" izz="${izz}" />
+      </inertial>
+      <collision>
+        <origin rpy="${origin_rpy}" xyz="${origin_xyz}" />
+        <geometry>
+          <mesh filename="${meshfile}" scale="1 1 1"/>
+        </geometry>
+      </collision>
+      <visual>
+        <origin rpy="${origin_rpy}" xyz="${origin_xyz}" />
+        <geometry>
+          <mesh filename="${meshfile}" scale="1 1 1"/>
+        </geometry>
+        <material name="red">
+          <color rgba="1.0 0.0 0.0 1.0"/>
+        </material>
+      </visual>
+    </link>
+    <gazebo reference="${name}">
+        <material>Gazebo/WhiteGlow</material>
+    </gazebo>
+ </xacro:macro>
  <xacro:macro name="create_noa" params="name origin_rpy origin_xyz parent">
   <link name="${name}">

Commit message: Se implementan los .stl del tornillo y la tuerca y se valida que la tuerca pueda ser insertada en el tornillo

File: proyecto_intermedio_robotica/urdf/links_joints.xacro (robot description, xacro)
@@ -64,7 +64,7 @@
     </link>
     <gazebo reference="${name}">
-      <mu1>10000.0</mu1>
-      <mu2>10000.0</mu2>
-      <minDepth>0.03</minDepth>
+      <mu1>100.0</mu1>
+      <mu2>100.0</mu2>
+      <minDepth>0.003</minDepth>
       <maxVel>0</maxVel>
         <!--<material>Gazebo/WhiteGlow</material>-->

File: proyecto_intermedio_robotica/urdf/tuerca.xacro (robot description, xacro)
@@ -1,14 +1,14 @@
 <?xml version="1.0"?>
-<robot name="tornillo_robot">
-     <link name="tornillo">
+<robot name="tuerca_robot">
+     <link name="tuerca">
       <inertial>
-        <mass value="0.01895747" />
+        <mass value="0.00325529" />
         <origin rpy="0.0 0.0 0.0" xyz="0.0 0.0 0.0" />
-        <inertia ixx="0.00000280" ixy="0.0" ixz="0.0" iyy="0.00000280" iyz="0.0" izz="0.00000024" />
+        <inertia ixx="0.00000007" ixy="0.0" ixz="0.0" iyy="0.00000007" iyz="0.0" izz="0.00000012" />
       </inertial>
       <collision>
         <origin rpy="0.0 0.0 0.0" xyz="0.0 0.0 0.0" />
         <geometry>
-          <mesh filename="package://proyecto_intermedio_robotica/meshes/tornillo_colision.stl" scale="0.01 0.01 0.01"/>
+          <mesh filename="package://proyecto_intermedio_robotica/meshes/tuerca_colision.stl" scale="0.01 0.01 0.01"/>
         </geometry>
       </collision>
@@ -16,5 +16,5 @@
         <origin rpy="0.0 0.0 0.0" xyz="0.0 0.0 0.0" />
         <geometry>
-          <mesh filename="package://proyecto_intermedio_robotica/meshes/tornillo.stl" scale="0.01 0.01 0.01"/>
+          <mesh filename="package://proyecto_intermedio_robotica/meshes/tuerca.stl" scale="0.01 0.01 0.01"/>
         </geometry>
         <material name="red">
@@ -23,5 +23,5 @@
       </visual>
     </link>
-    <gazebo reference="tornillo">
+    <gazebo reference="tuerca">
       <mu1>10.0</mu1>
       <mu2>10.0</mu2>
