Commit message: Se implementa el control del robot por esfuerzos y fricciónentre las superficies, se valida funcionamiento del gripper satisfactoriamente

File: proyecto_intermedio_robotica/urdf/4r_robot_gazebo.xacro (robot description, xacro)
@@ -23,5 +23,5 @@
      origin_rpy="0 0 -1.5708" origin_xyz="0 0 0.094375"
      parent="${link_00_name}" child="link_1"
-     limit_e="10" limit_l="-3.14" limit_u="3.14" limit_v="5.0"
+     limit_e="100" limit_l="-3.14" limit_u="3.14" limit_v="0.5"
      />
      <xacro:m_link_mesh name="link_1"
@@ -39,5 +39,5 @@
      origin_rpy="1.5708 -1.5708 1.5708" origin_xyz="0 0 0.0415"
      parent="link_1" child="link_2"
-     limit_e="10" limit_l="-3.14" limit_u="3.14" limit_v="5.0"
+     limit_e="100" limit_l="-3.14" limit_u="3.14" limit_v="0.5"
      />
      <xacro:m_link_mesh name="link_2"
@@ -55,5 +55,5 @@
      origin_rpy="0 0 0" origin_xyz="0.107 0 0"
      parent="link_2" child="link_3"
-     limit_e="10" limit_l="-3.14" limit_u="3.14" limit_v="5.0"
+     limit_e="100" limit_l="-3.14" limit_u="3.14" limit_v="0.5"
      />
      <xacro:m_link_mesh name="link_3"
@@ -71,5 +71,5 @@
      origin_rpy="0 0 0" origin_xyz="0.107 0 0"
      parent="link_3" child="link_4"
-     limit_e="10" limit_l="-3.14" limit_u="3.14" limit_v="5.0"
+     limit_e="100" limit_l="-3.14" limit_u="3.14" limit_v="0.5"
      />
      <xacro:m_link_mesh name="link_4"
@@ -87,5 +87,5 @@
      origin_rpy="0 0 0" origin_xyz="0.088 0.0001 -0.04"
      parent="link_4" child="finger_1"
-     limit_e="10" limit_l="0" limit_u="0.02" limit_v="5.0"
+     limit_e="10000" limit_l="0" limit_u="0.02" limit_v="0.5"
      />
      <xacro:m_link_mesh name="finger_1"
@@ -103,5 +103,5 @@
      origin_rpy="3.1416 0 0" origin_xyz="0.088 -0.0001 0.04"
      parent="link_4" child="finger_2"
-     limit_e="10" limit_l="0" limit_u="0.02" limit_v="5.0"
+     limit_e="10000" limit_l="0" limit_u="0.02" limit_v="0.5"
      mimic_joint="gripper_1" m_multiplier="1" m_offset="0"
      />

File: proyecto_intermedio_robotica/urdf/Objeto.xacro (robot description, xacro)
@@ -18,15 +18,11 @@
          </geometry>
        </collision>
-       <surface>
-          <friction>
-           <ode>
-            <mu>10</mu>
-            <mu2>10</mu2>
-           </ode>
-          </friction>
-        </surface>
      </link>
      <gazebo reference="my_box">
-       <material>Gazebo/Blue</material>
+      <mu1>10000.0</mu1>
+      <mu2>10000.0</mu2>
+      <minDepth>0.03</minDepth>
+      <maxVel>0</maxVel>
+      <material>Gazebo/Blue</material>
      </gazebo>
 </robot>

File: proyecto_intermedio_robotica/urdf/links_joints.xacro (robot description, xacro)
@@ -12,8 +12,8 @@
 	      <type>transmission_interface/SimpleTransmission</type>
 	      <joint name="${name}">
-		<hardwareInterface>hardware_interface/PositionJointInterface</hardwareInterface>
+		<hardwareInterface>hardware_interface/EffortJointInterface</hardwareInterface>
 	      </joint>
 	      <actuator name="motor_${name}">
-		<hardwareInterface>hardware_interface/PositionJointInterface</hardwareInterface>
+		<hardwareInterface>hardware_interface/EffortJointInterface</hardwareInterface>
 		<mechanicalReduction>1</mechanicalReduction>
 	      </actuator>
@@ -32,8 +32,8 @@
       <type>transmission_interface/SimpleTransmission</type>
       <joint name="${name}">
-  <hardwareInterface>hardware_interface/PositionJointInterface</hardwareInterface>
+  <hardwareInterface>hardware_interface/EffortJointInterface</hardwareInterface>
       </joint>
       <actuator name="motor_${name}">
-  <hardwareInterface>hardware_interface/PositionJointInterface</hardwareInterface>
+  <hardwareInterface>hardware_interface/EffortJointInterface</hardwareInterface>
   <mechanicalReduction>1</mechanicalReduction>
       </actuator>
@@ -64,4 +64,8 @@
     </link>
     <gazebo reference="${name}">
+      <mu1>10000.0</mu1>
+      <mu2>10000.0</mu2>
+      <minDepth>0.03</minDepth>
+      <maxVel>0</maxVel>
         <!--<material>Gazebo/WhiteGlow</material>-->
         <material>Gazebo/BlackTransparent</material>
@@ -95,4 +99,41 @@
     </gazebo>
  </xacro:macro>
+  <xacro:macro name="link_mesh_2" params="name origin_xyz origin_rpy meshfile mass ixx ixy ixz iyy iyz izz">
+    <link name="${name}">
+      <inertial>
+        <mass value="${mass}" />
+        <origin rpy="${origin_rpy}" xyz="${origin_xyz}" />
+        <inertia ixx="${ixx}" ixy="${ixy}" ixz="${ixz}" iyy="${iyy}" iyz="${iyz}" izz="${izz}" />
+      </inertial>
+      <collision>
+        <origin rpy="${origin_rpy}" xyz="${origin_xyz}" />
+        <geometry>
+          <mesh filename="${meshfile}" scale="1 1 1"/>
+        </geometry>
+      </collision>
+      <visual>
+        <origin rpy="${origin_rpy}" xyz="${origin_xyz}" />
+        <geometry>
+          <mesh filename="${meshfile}" scale="1 1 1"/>
+        </geometry>
+        <material name="red">
+          <color rgba="1.0 0.0 0.0 1.0"/>
+        </material>
+      </visual>
+      <surface>
+          <friction>
+           <ode>
+            <mu>1000</mu>
+            <mu2>1000</mu2>
+            <minDepth>0.003</minDepth>
+            <maxVel>0</maxVel>
+           </ode>
+          </friction>
+        </surface>
+    </link>
+    <gazebo reference="${name}">
+        <material>Gazebo/WhiteGlow</material>
+    </gazebo>
+ </xacro:macro>
  <xacro:macro name="create_noa" params="name origin_rpy origin_xyz parent">
   <link name="${name}">

Commit message: Se soluciona la vibración en el movimiento del robot con la implementación de un controlador hybrido

File: proyecto_intermedio_robotica/urdf/4r_robot_gazebo.xacro (robot description, xacro)
@@ -23,5 +23,5 @@
      origin_rpy="0 0 -1.5708" origin_xyz="0 0 0.094375"
      parent="${link_00_name}" child="link_1"
-     limit_e="50" limit_l="-3.14" limit_u="3.14" limit_v="0.5"
+     limit_e="50" limit_l="-3.14" limit_u="3.14" limit_v="5"
      />
      <xacro:m_link_mesh name="link_1"
@@ -39,5 +39,5 @@
      origin_rpy="1.5708 -1.5708 1.5708" origin_xyz="0 0 0.0415"
      parent="link_1" child="link_2"
-     limit_e="50" limit_l="-3.14" limit_u="3.14" limit_v="0.5"
+     limit_e="50" limit_l="-3.14" limit_u="3.14" limit_v="5"
      />
      <xacro:m_link_mesh name="link_2"
@@ -55,5 +55,5 @@
      origin_rpy="0 0 0" origin_xyz="0.107 0 0"
      parent="link_2" child="link_3"
-     limit_e="50" limit_l="-3.14" limit_u="3.14" limit_v="0.5"
+     limit_e="50" limit_l="-3.14" limit_u="3.14" limit_v="5"
      />
      <xacro:m_link_mesh name="link_3"
@@ -71,5 +71,5 @@
      origin_rpy="0 0 0" origin_xyz="0.107 0 0"
      parent="link_3" child="link_4"
-     limit_e="50" limit_l="-3.14" limit_u="3.14" limit_v="0.5"
+     limit_e="50" limit_l="-3.14" limit_u="3.14" limit_v="5"
      />
      <xacro:m_link_mesh name="link_4"
@@ -82,5 +82,5 @@
      izz="0.00002116"
      />
-     <xacro:m_joint name="gripper_1"
+     <xacro:m_joint_effort name="gripper_1"
      type="prismatic"
      axis_xyz="0 0 1"

File: proyecto_intermedio_robotica/urdf/links_joints.xacro (robot description, xacro)
@@ -2,4 +2,23 @@
 <robot xmlns:xacro="http://www.ros.org/wiki/xacro">
  <xacro:macro name="m_joint" params="name type axis_xyz origin_rpy origin_xyz parent child limit_e limit_l limit_u limit_v">
+    <joint name="${name}" type="${type}">
+      <axis xyz="${axis_xyz}" />
+      <limit effort="${limit_e}" lower="${limit_l}" upper="${limit_u}" velocity="${limit_v}" />
+      <origin rpy="${origin_rpy}" xyz="${origin_xyz}" />
+      <parent link="${parent}" />
+      <child link="${child}" />
+    </joint>
+	<transmission name="trans_${name}">
+	      <type>transmission_interface/SimpleTransmission</type>
+	      <joint name="${name}">
+		<hardwareInterface>hardware_interface/PositionJointInterface</hardwareInterface>
+	      </joint>
+	      <actuator name="motor_${name}">
+		<hardwareInterface>hardware_interface/PositionJointInterface</hardwareInterface>
+		<mechanicalReduction>1</mechanicalReduction>
+	      </actuator>
+	    </transmission>
+ </xacro:macro>
+  <xacro:macro name="m_joint_effort" params="name type axis_xyz origin_rpy origin_xyz parent child limit_e limit_l limit_u limit_v">
     <joint name="${name}" type="${type}">
       <axis xyz="${axis_xyz}" />

Commit message: Add files via upload

File: proyecto_intermedio_robotica/urdf/4r_robot_gazebo.xacro (robot description, xacro)
@@ -23,5 +23,5 @@
      origin_rpy="0 0 -1.5708" origin_xyz="0 0 0.094375"
      parent="${link_00_name}" child="link_1"
-     limit_e="50" limit_l="-3.14" limit_u="3.14" limit_v="5"
+     limit_e="100" limit_l="-3.14" limit_u="3.14" limit_v="0.5"
      />
      <xacro:m_link_mesh name="link_1"
@@ -39,5 +39,5 @@
      origin_rpy="1.5708 -1.5708 1.5708" origin_xyz="0 0 0.0415"
      parent="link_1" child="link_2"
-     limit_e="50" limit_l="-3.14" limit_u="3.14" limit_v="5"
+     limit_e="100" limit_l="-3.14" limit_u="3.14" limit_v="0.5"
      />
      <xacro:m_link_mesh name="link_2"
@@ -55,5 +55,5 @@
      origin_rpy="0 0 0" origin_xyz="0.107 0 0"
      parent="link_2" child="link_3"
-     limit_e="50" limit_l="-3.14" limit_u="3.14" limit_v="5"
+     limit_e="100" limit_l="-3.14" limit_u="3.14" limit_v="0.5"
      />
      <xacro:m_link_mesh name="link_3"
@@ -71,5 +71,5 @@
      origin_rpy="0 0 0" origin_xyz="0.107 0 0"
      parent="link_3" child="link_4"
-     limit_e="50" limit_l="-3.14" limit_u="3.14" limit_v="5"
+     limit_e="100" limit_l="-3.14" limit_u="3.14" limit_v="0.5"
      />
      <xacro:m_link_mesh name="link_4"
@@ -82,10 +82,10 @@
      izz="0.00002116"
      />
-     <xacro:m_joint_effort name="gripper_1"
+     <xacro:m_joint name="gripper_1"
      type="prismatic"
      axis_xyz="0 0 1"
      origin_rpy="0 0 0" origin_xyz="0.088 0.0001 -0.04"
      parent="link_4" child="finger_1"
-     limit_e="50" limit_l="0" limit_u="0.02" limit_v="0.05"
+     limit_e="10000" limit_l="0" limit_u="0.02" limit_v="0.5"
      />
      <xacro:m_link_mesh name="finger_1"
@@ -103,6 +103,6 @@
      origin_rpy="3.1416 0 0" origin_xyz="0.088 -0.0001 0.04"
      parent="link_4" child="finger_2"
-     limit_e="50" limit_l="0" limit_u="0.02" limit_v="0.05"
-     mimic_joint="gripper_1" m_multiplier="5" m_offset="0"
+     limit_e="10000" limit_l="0" limit_u="0.02" limit_v="0.5"
+     mimic_joint="gripper_1" m_multiplier="1" m_offset="0"
      />
      <xacro:m_link_mesh name="finger_2"

File: proyecto_intermedio_robotica/urdf/cubo1.xacro (robot description, xacro)
@@ -1,14 +1,14 @@
 <?xml version="1.0"?>
-<robot name="tornillo_robot">
-     <link name="tornillo">
+<robot name="cubo1_robot">
+     <link name="cubo1">
       <inertial>
-        <mass value="0.01895747" />
+        <mass value="0.0981" />
         <origin rpy="0.0 0.0 0.0" xyz="0.0 0.0 0.0" />
-        <inertia ixx="0.00000280" ixy="0.0" ixz="0.0" iyy="0.00000280" iyz="0.0" izz="0.00000024" />
+        <inertia ixx="0.1476" ixy="0.0" ixz="0.0" iyy="0.1476" iyz="0.0" izz="0.0590" />
       </inertial>
       <collision>
         <origin rpy="0.0 0.0 0.0" xyz="0.0 0.0 0.0" />
         <geometry>
-          <mesh filename="package://proyecto_intermedio_robotica/meshes/tornillo_colision.stl" scale="0.01 0.01 0.01"/>
+          <mesh filename="package://proyecto_intermedio_robotica/meshes/Cubito.stl" scale="0.01 0.01 0.01"/>
         </geometry>
       </collision>
@@ -16,5 +16,5 @@
         <origin rpy="0.0 0.0 0.0" xyz="0.0 0.0 0.0" />
         <geometry>
-          <mesh filename="package://proyecto_intermedio_robotica/meshes/tornillo.stl" scale="0.01 0.01 0.01"/>
+          <mesh filename="package://proyecto_intermedio_robotica/meshes/Cubito.stl" scale="0.01 0.01 0.01"/>
         </geometry>
         <material name="red">
@@ -23,11 +23,10 @@
       </visual>
     </link>
-    <gazebo reference="tornillo">
+    <gazebo reference="cubo1">
       <mu1>10.0</mu1>
       <mu2>10.0</mu2>
       <minDepth>0.003</minDepth>
       <maxVel>0</maxVel>
-        <material>Gazebo/<color rgba="0.0 1.0 0.0 0.0"/>
-        </material>
+        <material>Gazebo/Blue</material>
     </gazebo>
 </robot>

File: proyecto_intermedio_robotica/urdf/cubo2.xacro (robot description, xacro)
@@ -1,14 +1,14 @@
 <?xml version="1.0"?>
-<robot name="tornillo_robot">
-     <link name="tornillo">
+<robot name="cubo2_robot">
+     <link name="cubo2">
       <inertial>
-        <mass value="0.01895747" />
+        <mass value="0.0567" />
         <origin rpy="0.0 0.0 0.0" xyz="0.0 0.0 0.0" />
-        <inertia ixx="0.00000280" ixy="0.0" ixz="0.0" iyy="0.00000280" iyz="0.0" izz="0.00000024" />
+        <inertia ixx="0.0193" ixy="0.0" ixz="0.0" iyy="0.0193" iyz="0.0" izz="0.0237" />
       </inertial>
       <collision>
         <origin rpy="0.0 0.0 0.0" xyz="0.0 0.0 0.0" />
         <geometry>
-          <mesh filename="package://proyecto_intermedio_robotica/meshes/tornillo_colision.stl" scale="0.01 0.01 0.01"/>
+          <mesh filename="package://proyecto_intermedio_robotica/meshes/Cubitofake.stl" scale="0.01 0.01 0.01"/>
         </geometry>
       </collision>
@@ -16,5 +16,5 @@
         <origin rpy="0.0 0.0 0.0" xyz="0.0 0.0 0.0" />
         <geometry>
-          <mesh filename="package://proyecto_intermedio_robotica/meshes/tornillo.stl" scale="0.01 0.01 0.01"/>
+          <mesh filename="package://proyecto_intermedio_robotica/meshes/Cubitofake.stl" scale="0.01 0.01 0.01"/>
         </geometry>
         <material name="red">
@@ -23,11 +23,10 @@
       </visual>
     </link>
-    <gazebo reference="tornillo">
+    <gazebo reference="cubo2">
       <mu1>10.0</mu1>
       <mu2>10.0</mu2>
       <minDepth>0.003</minDepth>
       <maxVel>0</maxVel>
-        <material>Gazebo/<color rgba="0.0 1.0 0.0 0.0"/>
-        </material>
+        <material>Gazebo/Blue</material>
     </gazebo>
 </robot>

File: proyecto_intermedio_robotica/urdf/links_joints.xacro (robot description, xacro)
@@ -2,23 +2,4 @@
 <robot xmlns:xacro="http://www.ros.org/wiki/xacro">
  <xacro:macro name="m_joint" params="name type axis_xyz origin_rpy origin_xyz parent child limit_e limit_l limit_u limit_v">
-    <joint name="${name}" type="${type}">
-      <axis xyz="${axis_xyz}" />
-      <limit effort="${limit_e}" lower="${limit_l}" upper="${limit_u}" velocity="${limit_v}" />
-      <origin rpy="${origin_rpy}" xyz="${origin_xyz}" />
-      <parent link="${parent}" />
-      <child link="${child}" />
-    </joint>
-	<transmission name="trans_${name}">
-	      <type>transmission_interface/SimpleTransmission</type>
-	      <joint name="${name}">
-		<hardwareInterface>hardware_interface/PositionJointInterface</hardwareInterface>
-	      </joint>
-	      <actuator name="motor_${name}">
-		<hardwareInterface>hardware_interface/PositionJointInterface</hardwareInterface>
-		<mechanicalReduction>1</mechanicalReduction>
-	      </actuator>
-	    </transmission>
- </xacro:macro>
-  <xacro:macro name="m_joint_effort" params="name type axis_xyz origin_rpy origin_xyz parent child limit_e limit_l limit_u limit_v">
     <joint name="${name}" type="${type}">
       <axis xyz="${axis_xyz}" />

File: proyecto_intermedio_robotica/urdf/tuerca.xacro (robot description, xacro)
@@ -10,5 +10,5 @@
         <origin rpy="0.0 0.0 0.0" xyz="0.0 0.0 0.0" />
         <geometry>
-          <mesh filename="package://proyecto_intermedio_robotica/meshes/tuerca_colision_2.stl" scale="0.01 0.01 0.01"/>
+          <mesh filename="package://proyecto_intermedio_robotica/meshes/tuerca_colision.stl" scale="0.01 0.01 0.01"/>
         </geometry>
       </collision>
@@ -28,5 +28,6 @@
       <minDepth>0.003</minDepth>
       <maxVel>0</maxVel>
-        <material>Gazebo/Blue</material>
+        <material>Gazebo/<color rgba="0.0 1.0 0.0 0.0"/>
+        </material>
     </gazebo>
 </robot>

Commit message: Se avanza en los puntos de los robots y en los servicios de gazebo_ros

File: proyecto_intermedio_robotica/urdf/4r_robot_gazebo.xacro (robot description, xacro)
@@ -87,5 +87,5 @@
      origin_rpy="0 0 0" origin_xyz="0.088 0.0001 -0.04"
      parent="link_4" child="finger_1"
-     limit_e="2.5" limit_l="0" limit_u="0.02" limit_v="5.0"
+     limit_e="2" limit_l="0" limit_u="0.02" limit_v="5.0"
      />
      <xacro:m_link_mesh name="finger_1"
@@ -103,5 +103,5 @@
      origin_rpy="3.1416 0 0" origin_xyz="0.088 -0.0001 0.04"
      parent="link_4" child="finger_2"
-     limit_e="2.5" limit_l="0" limit_u="0.02" limit_v="5.0"
+     limit_e="2" limit_l="0" limit_u="0.02" limit_v="5.0"
      mimic_joint="gripper_1" m_multiplier="5" m_offset="0"
      />

File: proyecto_intermedio_robotica/urdf/tornillo.xacro (robot description, xacro)
@@ -4,5 +4,5 @@
       <inertial>
         <mass value="0.01895747" />
-        <origin rpy="0.0 0.0 0.0" xyz="0.0 0.0 0.0" />
+        <origin rpy="0.0 0.0 0.0" xyz="0.0 0.0 0.0025" />
         <inertia ixx="0.00000280" ixy="0.0" ixz="0.0" iyy="0.00000280" iyz="0.0" izz="0.00000024" />
       </inertial>

Commit message: Se finaliza las trayectorias para el ensamble de los 6 modelos satisfactoriamente

File: proyecto_intermedio_robotica/urdf/4r_robot_gazebo.xacro (robot description, xacro)
@@ -89,5 +89,5 @@
      limit_e="2" limit_l="0" limit_u="0.02" limit_v="5.0"
      />
-     <xacro:m_link_mesh name="finger_1"
+     <xacro:m_link_mesh_2 name="finger_1"
      origin_xyz="0 0 0"
      origin_rpy="0 0 0"
@@ -106,5 +106,5 @@
      mimic_joint="gripper_1" m_multiplier="5" m_offset="0"
      />
-     <xacro:m_link_mesh name="finger_2"
+     <xacro:m_link_mesh_2 name="finger_2"
      origin_xyz="0 0 0"
      origin_rpy="0 0 0"

File: proyecto_intermedio_robotica/urdf/links_joints.xacro (robot description, xacro)
@@ -91,5 +91,5 @@
     </gazebo>
  </xacro:macro>
- <xacro:macro name="link_mesh" params="name origin_xyz origin_rpy meshfile mass ixx ixy ixz iyy iyz izz">
+ <xacro:macro name="m_link_mesh_2" params="name origin_xyz origin_rpy meshfile mass ixx ixy ixz iyy iyz izz">
     <link name="${name}">
       <inertial>
@@ -98,59 +98,21 @@
         <inertia ixx="${ixx}" ixy="${ixy}" ixz="${ixz}" iyy="${iyy}" iyz="${iyz}" izz="${izz}" />
       </inertial>
-      <collision>
-        <origin rpy="${origin_rpy}" xyz="${origin_xyz}" />
-        <geometry>
-          <mesh filename="${meshfile}" scale="1 1 1"/>
-        </geometry>
-      </collision>
       <visual>
         <origin rpy="${origin_rpy}" xyz="${origin_xyz}" />
         <geometry>
-          <mesh filename="${meshfile}" scale="1 1 1"/>
+          <mesh filename="${meshfile}" scale="0.1 0.1 0.1"/>
         </geometry>
-        <material name="red">
-          <color rgba="1.0 0.0 0.0 1.0"/>
+        <material name="Cyan">
+          <color rgba="0 1.0 1.0 1.0"/>
         </material>
       </visual>
     </link>
     <gazebo reference="${name}">
-        <material>Gazebo/WhiteGlow</material>
-    </gazebo>
- </xacro:macro>
-  <xacro:macro name="link_mesh_2" params="name origin_xyz origin_rpy meshfile mass ixx ixy ixz iyy iyz izz">
-    <link name="${name}">
-      <inertial>
-        <mass value="${mass}" />
-        <origin rpy="${origin_rpy}" xyz="${origin_xyz}" />
-        <inertia ixx="${ixx}" ixy="${ixy}" ixz="${ixz}" iyy="${iyy}" iyz="${iyz}" izz="${izz}" />
-      </inertial>
-      <collision>
-        <origin rpy="${origin_rpy}" xyz="${origin_xyz}" />
-        <geometry>
-          <mesh filename="${meshfile}" scale="1 1 1"/>
-        </geometry>
-      </collision>
-      <visual>
-        <origin rpy="${origin_rpy}" xyz="${origin_xyz}" />
-        <geometry>
-          <mesh filename="${meshfile}" scale="1 1 1"/>
-        </geometry>
-        <material name="red">
-          <color rgba="1.0 0.0 0.0 1.0"/>
-        </material>
-      </visual>
-      <surface>
-          <friction>
-           <ode>
-            <mu>1000</mu>
-            <mu2>1000</mu2>
-            <minDepth>0.003</minDepth>
-            <maxVel>0</maxVel>
-           </ode>
-          </friction>
-        </surface>
-    </link>
-    <gazebo reference="${name}">
-        <material>Gazebo/WhiteGlow</material>
+      <mu1>100.0</mu1>
+      <mu2>100.0</mu2>
+      <minDepth>0.003</minDepth>
+      <maxVel>0</maxVel>
+        <!--<material>Gazebo/WhiteGlow</material>-->
+        <material>Gazebo/BlackTransparent</material>
     </gazebo>
  </xacro:macro>

File: proyecto_intermedio_robotica/urdf/tornillo.xacro (robot description, xacro)
@@ -24,4 +24,5 @@
     </link>
     <gazebo reference="tornillo">
+      <turnGravityOff>true</turnGravityOff>
       <mu1>100.0</mu1>
       <mu2>100.0</mu2>

File: proyecto_intermedio_robotica/urdf/tuerca.xacro (robot description, xacro)
@@ -3,5 +3,5 @@
      <link name="tuerca">
       <inertial>
-        <mass value="0.00325529" />
+        <mass value="0.00001" />
         <origin rpy="0.0 0.0 0.0" xyz="0.0 0.0 0.0" />
         <inertia ixx="0.00000007" ixy="0.0" ixz="0.0" iyy="0.00000007" iyz="0.0" izz="0.00000012" />
