Commit message: Se modifican los solidos de colisión del tornillo y de la tuerca

File: proyecto_intermedio_robotica/urdf/tornillo.xacro (robot description, xacro)
@@ -10,5 +10,5 @@
         <origin rpy="0.0 0.0 0.0" xyz="0.0 0.0 0.0" />
         <geometry>
-          <mesh filename="package://proyecto_intermedio_robotica/meshes/tornillo_colision.stl" scale="0.01 0.01 0.01"/>
+          <mesh filename="package://proyecto_intermedio_robotica/meshes/tornillo_colision_2.stl" scale="0.01 0.01 0.01"/>
         </geometry>
       </collision>

File: proyecto_intermedio_robotica/urdf/tuerca.xacro (robot description, xacro)
@@ -10,5 +10,5 @@
         <origin rpy="0.0 0.0 0.0" xyz="0.0 0.0 0.0" />
         <geometry>
-          <mesh filename="package://proyecto_intermedio_robotica/meshes/tuerca_colision.stl" scale="0.01 0.01 0.01"/>
+          <mesh filename="package://proyecto_intermedio_robotica/meshes/tuerca_colision_2.stl" scale="0.01 0.01 0.01"/>
         </geometry>
       </collision>

Commit message: Se implementa y valida la trayectoría para recojer y ensamblar tuerca_1 y tornillo_1

File: proyecto_intermedio_robotica/urdf/tornillo.xacro (robot description, xacro)
@@ -4,5 +4,5 @@
       <inertial>
         <mass value="0.01895747" />
-        <origin rpy="0.0 0.0 0.0" xyz="0.0 0.0 0.0025" />
+        <origin rpy="0.0 0.0 0.0" xyz="0.0 0.0 0.0" />
         <inertia ixx="0.00000280" ixy="0.0" ixz="0.0" iyy="0.00000280" iyz="0.0" izz="0.00000024" />
       </inertial>

File: proyecto_intermedio_robotica/urdf/tuerca.xacro (robot description, xacro)
@@ -28,5 +28,5 @@
       <minDepth>0.003</minDepth>
       <maxVel>0</maxVel>
-        <material>Gazebo/Blue</material>
+        <material>Gazebo/Red</material>
     </gazebo>
 </robot>

Commit message: SE implementan las zonas marcadas para los objetos y se valida su correcto funcionamiento

File: proyecto_intermedio_robotica/urdf/tornillo.xacro (robot description, xacro)
@@ -29,5 +29,5 @@
       <minDepth>0.003</minDepth>
       <maxVel>0</maxVel>
-        <material>Gazebo/Blue</material>
+        <material>Gazebo/BlueTransparentOverlay</material>
     </gazebo>
 </robot>

File: proyecto_intermedio_robotica/urdf/tuerca.xacro (robot description, xacro)
@@ -28,5 +28,5 @@
       <minDepth>0.003</minDepth>
       <maxVel>0</maxVel>
-        <material>Gazebo/Red</material>
+        <material>Gazebo/RedTransparentOverlay</material>
     </gazebo>
 </robot>
